File: speaker-lights.brd (EAGLE design)
At the start: 160 x 100 mm, 2 parts

Commit message: start project
Parts:
- moved INPUT 152.6 mm to (129.0, 37.1), turned to 180 degrees
- moved OUTPUT 70.1 mm to (13.2, 38.1)
Connections:
- net N$1 renamed LOUTSW
- net N$2 renamed ROUTSW
- new net LINSW: INPUT.4
- new net RINSW: INPUT.3
Routing:
- net LCHAN: track 0.00 -> 131.6 mm
- net RCHAN: track 0.00 -> 114.6 mm
- added copper zone on layer 16, net GND
Other:
- board size 160 x 100 mm -> 140 x 68.1 mm
Changed lines of the file:
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@@
 <setting verticaltext="up"/>
 </settings>
-<grid distance="50" unitdist="mil" unit="mil" style="lines" multiple="1" display="no" altdistance="5" altunitdist="mil" altunit="mil"/>
+<grid distance="10" unitdist="mil" unit="mil" style="dots" multiple="1" display="yes" altdistance="5" altunitdist="mil" altunit="mil"/>
 <layers>
 <layer number="1" name="Top" color="4" fill="1" visible="yes" active="yes"/>
@@
 <board>
 <plain>
-<wire x1="0" y1="0" x2="160" y2="0" width="0" layer="20"/>
-<wire x1="160" y1="0" x2="160" y2="100" width="0" layer="20"/>
-<wire x1="160" y1="100" x2="0" y2="100" width="0" layer="20"/>
-<wire x1="0" y1="100" x2="0" y2="0" width="0" layer="20"/>
+<wire x1="0" y1="0" x2="139.954" y2="0" width="0" layer="20"/>
+<wire x1="139.954" y1="0" x2="139.954" y2="67.818" width="0" layer="20"/>
+<wire x1="139.954" y1="67.818" x2="0" y2="68.072" width="0" layer="20"/>
+<wire x1="0" y1="68.072" x2="0" y2="0" width="0" layer="20"/>
 </plain>
 <attributes>
@@
 </autorouter>
 <elements>
-<element name="INPUT" library="con-hirschmann" library_urn="urn:adsk.eagle:library:153" package="PG203J" package3d_urn="urn:adsk.eagle:package:7447/1" value="PG203J" x="-16.51" y="-8.89" smashed="yes">
-<attribute name="MF" value="" x="-16.51" y="-8.89" size="1.778" layer="27" display="off"/>
-<attribute name="MPN" value="" x="-16.51" y="-8.89" size="1.778" layer="27" display="off"/>
-<attribute name="NAME" x="-22.225" y="-2.54" size="1.27" layer="25" ratio="10"/>
-<attribute name="OC_FARNELL" value="unknown" x="-16.51" y="-8.89" size="1.778" layer="27" display="off"/>
-<attribute name="OC_NEWARK" value="unknown" x="-16.51" y="-8.89" size="1.778" layer="27" display="off"/>
-<attribute name="POPULARITY" value="6" x="-16.51" y="-8.89" size="1.778" layer="27" display="off"/>
-<attribute name="VALUE" x="-22.86" y="-16.51" size="1.27" layer="27" ratio="10"/>
+<element name="INPUT" library="con-hirschmann" library_urn="urn:adsk.eagle:library:153" package="PG203J" package3d_urn="urn:adsk.eagle:package:7447/1" value="PG203J" x="129.032" y="37.084" smashed="yes" rot="R180">
+<attribute name="MF" value="" x="129.032" y="37.084" size="1.778" layer="27" rot="R180" display="off"/>
+<attribute name="MPN" value="" x="129.032" y="37.084" size="1.778" layer="27" rot="R180" display="off"/>
+<attribute name="NAME" x="134.747" y="30.734" size="1.27" layer="25" ratio="10" rot="R180"/>
+<attribute name="OC_FARNELL" value="unknown" x="129.032" y="37.084" size="1.778" layer="27" rot="R180" display="off"/>
+<attribute name="OC_NEWARK" value="unknown" x="129.032" y="37.084" size="1.778" layer="27" rot="R180" display="off"/>
+<attribute name="POPULARITY" value="6" x="129.032" y="37.084" size="1.778" layer="27" rot="R180" display="off"/>
+<attribute name="VALUE" x="135.382" y="44.704" size="1.27" layer="27" ratio="10" rot="R180"/>
 </element>
-<element name="OUTPUT" library="con-hirschmann" library_urn="urn:adsk.eagle:library:153" package="PG203J" package3d_urn="urn:adsk.eagle:package:7447/1" value="PG203J" x="-16.51" y="-25.4" smashed="yes">
-<attribute name="MF" value="" x="-16.51" y="-25.4" size="1.778" layer="27" display="off"/>
-<attribute name="MPN" value="" x="-16.51" y="-25.4" size="1.778" layer="27" display="off"/>
-<attribute name="NAME" x="-22.225" y="-19.05" size="1.27" layer="25" ratio="10"/>
-<attribute name="OC_FARNELL" value="unknown" x="-16.51" y="-25.4" size="1.778" layer="27" display="off"/>
-<attribute name="OC_NEWARK" value="unknown" x="-16.51" y="-25.4" size="1.778" layer="27" display="off"/>
-<attribute name="POPULARITY" value="6" x="-16.51" y="-25.4" size="1.778" layer="27" display="off"/>
-<attribute name="VALUE" x="-22.86" y="-33.02" size="1.27" layer="27" ratio="10"/>
+<element name="OUTPUT" library="con-hirschmann" library_urn="urn:adsk.eagle:library:153" package="PG203J" package3d_urn="urn:adsk.eagle:package:7447/1" value="PG203J" x="13.208" y="38.1" smashed="yes">
+<attribute name="MF" value="" x="13.208" y="38.1" size="1.778" layer="27" display="off"/>
+<attribute name="MPN" value="" x="13.208" y="38.1" size="1.778" layer="27" display="off"/>
+<attribute name="NAME" x="7.493" y="44.45" size="1.27" layer="25" ratio="10"/>
+<attribute name="OC_FARNELL" value="unknown" x="13.208" y="38.1" size="1.778" layer="27" display="off"/>
+<attribute name="OC_NEWARK" value="unknown" x="13.208" y="38.1" size="1.778" layer="27" display="off"/>
+<attribute name="POPULARITY" value="6" x="13.208" y="38.1" size="1.778" layer="27" display="off"/>
+<attribute name="VALUE" x="6.858" y="30.48" size="1.27" layer="27" ratio="10"/>
 </element>
 </elements>
@@
 <contactref element="OUTPUT" pad="5"/>
 <contactref element="INPUT" pad="5"/>
-<wire x1="-18.2626" y1="-13.7922" x2="-18.2626" y2="-30.3022" width="0" layer="19" extent="1-1"/>
+<wire x1="11.4554" y1="33.1978" x2="15.6972" y2="28.956" width="0.1524" layer="1"/>
+<wire x1="15.6972" y1="28.956" x2="126.492" y2="28.956" width="0.1524" layer="1"/>
+<wire x1="126.492" y1="28.956" x2="130.7846" y2="33.2486" width="0.1524" layer="1"/>
+<wire x1="130.7846" y1="33.2486" x2="130.7846" y2="41.9862" width="0.1524" layer="1"/>
 </signal>
 <signal name="GND">
 <contactref element="OUTPUT" pad="1"/>
 <contactref element="INPUT" pad="1"/>
-<wire x1="-21.5138" y1="-9.0932" x2="-21.5138" y2="-25.6032" width="0" layer="19" extent="1-1"/>
+<polygon width="0.1524" layer="16">
+<vertex x="6.096" y="37.846"/>
+<vertex x="6.096" y="2.54"/>
+<vertex x="136.144" y="2.54"/>
+<vertex x="136.144" y="65.278"/>
+<vertex x="6.096" y="65.278"/>
+</polygon>
 </signal>
 <signal name="RCHAN">
 <contactref element="OUTPUT" pad="2"/>
 <contactref element="INPUT" pad="2"/>
-<wire x1="-13.6652" y1="-3.9878" x2="-13.6652" y2="-20.4978" width="0" layer="19" extent="1-1"/>
-</signal>
-<signal name="N$1">
+<wire x1="16.0528" y1="43.0022" x2="26.8732" y2="32.1818" width="0.1524" layer="1"/>
+<wire x1="26.8732" y1="32.1818" x2="126.1872" y2="32.1818" width="0.1524" layer="1"/>
+</signal>
+<signal name="LOUTSW">
 <contactref element="OUTPUT" pad="4"/>
 </signal>
-<signal name="N$2">
+<signal name="ROUTSW">
 <contactref element="OUTPUT" pad="3"/>
 </signal>
+<signal name="LINSW">
+<contactref element="INPUT" pad="4"/>
+</signal>
+<signal name="RINSW">
+<contactref element="INPUT" pad="3"/>
+</signal>
 </signals>
